File: rotating_sphere_electronics/RS64c/LED_electronics.kicad_sch (KiCad schematic)
At the start: 17 parts, among them U401 STP24DP05BTR, U402 74HCT138

Commit message: R403, 404, 405 corrected
Parts:
- R403, R404, R405: LCSC C11702 -> C25099
Changed lines of the file:
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@@
 			)
 		)
-		(property "LCSC" "C11702"
+		(property "LCSC" "C25099"
 			(at 143.51 102.87 90)
 			(effects
@@
 			)
 		)
-		(property "LCSC" "C11702"
+		(property "LCSC" "C25099"
 			(at 143.51 107.95 90)
 			(effects
@@
 			)
 		)
-		(property "LCSC" "C11702"
+		(property "LCSC" "C25099"
 			(at 143.51 105.41 90)
 			(effects
